Commit message: yaml files added

File: src/wheel_time/urdf/wheel.urdf (robot description, URDF)
Before this commit: robot onshape, 2 links, 1 joints
Links:
- link wheel: mass 3.86134 -> 0.534374

Commit message: position rev controller added

File: src/wheel_time/urdf/wheel.urdf (robot description, URDF)
Before this commit: robot onshape, 2 links, 1 joints
Links:
- removed link base
- added link base_link, mass 11.195; collision mesh filename=file:///home/mackenzie/catkin_ws/src/wheel_time/urdf/base.s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; visual mesh filename=file:///home/mackenzie/catkin_ws/src/wheel_time/urdf/base.s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
- added link world
- link wheel: geometry collision mesh filename=file:///home/mackenzie/catkin_ws/src/wheel_time/urdf/wheel.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; visual mesh filename=file:///home/mackenzie/catkin_ws/src/wheel_time/urdf/wheel.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
Joints:
- added joint base_joint: type fixed, parent world, child base_link, origin xyz=0 0 0 rpy=0 0 0
- joint rev: child base -> wheel; origin xyz=-2.77556e-17 -8.67362e-18 0.2032 rpy=-1.5708 -0 0 -> xyz=-7.60623e-18 -3.5982e-17 0.2032 rpy=1.5708 -0.868659 3.14159; parent wheel -> base_link

Commit message: camera plugin added to urdf

File: src/wheel_time/urdf/wheel.urdf (robot description, URDF)
Before this commit: robot onshape, 3 links, 2 joints
Links:
- added link camera_link, mass 1e-5; collision box size=0.05 0.05 0.05; visual box size=0.05 0.05 0.05
Joints:
- added joint camera_joint: type fixed, parent world, child camera_link, origin xyz=0 1 .3 rpy=0 0 -1.57079632679, axis 1 0 0
